Commit message: Added mobiman_control pkg: control files for jackal_ur5. Updated mobiman_simulation: gazebo launch for sim and control tested successfully and visualized in rviz.

File: mobiman_simulation/urdf/jackal_fixedWheel.urdf.xacro (robot description, xacro)
@@ -3,5 +3,5 @@
   <xacro:property name="PI" value="3.1415926535897931" />
   <xacro:property name="wheelbase" value="0.262" />
-  <xacro:property name="track" value="0.38" /> <!--0.37559 NUA Note: Error:: MoveIt! collision matrix: "stack smashing detected"-->
+  <xacro:property name="track" value="0.38" />
   <xacro:property name="wheel_vertical_offset" value="0.0345" />
   <xacro:property name="footprint_vertical_offset" value="-0.0655" />
@@ -50,5 +50,5 @@
       <fdir1 value="1 0 0"/>
     </gazebo>
-    <joint name="${prefix}_wheel" type="fixed">
+    <joint name="${prefix}_wheel" type="continuous">
       <parent link="chassis_link"/>
       <child link="${prefix}_wheel_link" />
@@ -120,4 +120,5 @@
       </visual>
       <collision>
+        <!--origin xyz="0 0 0" rpy="0 0 0"/-->
         <geometry>
           <mesh filename="package://jackal_description/meshes/jackal-fender.stl"/>
@@ -135,4 +136,5 @@
       </visual>
       <collision>
+        <!--origin xyz="0 0 0" rpy="0 0 0"/-->
         <geometry>
           <mesh filename="package://jackal_description/meshes/accessory_fender.stl"/>
@@ -161,4 +163,5 @@
       </visual>
       <collision>
+        <!--origin xyz="0 0 0" rpy="0 0 0"/-->
         <geometry>
           <mesh filename="package://jackal_description/meshes/jackal-fender.stl"/>
@@ -176,4 +179,5 @@
       </visual>
       <collision>
+        <!--origin xyz="0 0 0" rpy="0 0 0"/-->
         <geometry>
           <mesh filename="package://jackal_description/meshes/accessory_fender.stl"/>

File: mobiman_simulation/urdf/jackal_fixedWheel_ur5.urdf.xacro (robot description, xacro)
@@ -1,22 +1,22 @@
 <?xml version="1.0" ?>
-<robot name="jackal_ur5" xmlns:xacro="http://www.ros.org/wiki/xacro">
-    <xacro:arg name="ns" default=""/>
-    <xacro:arg name="model" default=""/>
-    <!--xacro:property name="ns" value="$(arg ns)"/-->
-    <!--xacro:property name="arm_prefix" value="ur_arm_" /-->
-    <!--xacro:property name="path_meshes" value="package://tentabot/meshes" /-->
+<robot name="mobiman" xmlns:xacro="http://www.ros.org/wiki/xacro">
+    <xacro:arg name="robot_namespace" default="/"/>
+    <xacro:property name="arm_prefix" value="ur5_" />
+    <xacro:property name="path_meshes" value="package://mobiman_simulation/meshes" />
     <xacro:property name="M_PI" value="3.1415926535897931" />
     <xacro:property name="M_PI_2" value="1.570796327" />
-    <!-- Import macro for materials-->
-    <!--xacro:include filename="$(find tentabot)/urdf/materials.xacro" /-->
+    <xacro:include filename="$(find mobiman_simulation)/urdf/materials.xacro" />
     <!-- Import mobile base -->
-    <!--xacro:include filename="$(find turtlebot3_description)/urdf/turtlebot3_$(arg model)_with_ns.urdf.xacro"/-->
-    <!--xacro:include filename="$(find turtlebot3_description)/urdf/turtlebot3_$(arg model).urdf.xacro"/-->
     <!--xacro:include filename="$(find husky_description)/urdf/husky.urdf.xacro"/-->
     <xacro:include filename="$(find mobiman_simulation)/urdf/jackal_fixedWheel.urdf.xacro"/>
-    <!-- Import arm: UR5 -->
-    <xacro:include filename="$(find ur_description)/urdf/ur5.urdf.xacro"/>
-    <xacro:ur5_robot prefix="ur5_" joint_limited="true"/>
-    <!-- Create UR5 instance -->
+    <!-- Import robotic arm -->
+    <xacro:include filename="$(find ur_description)/urdf/inc/ur5_macro.xacro"/>
+    <xacro:ur5_robot prefix="${arm_prefix}" />
+    <!-- Import lidar-->
+    <!--xacro:include filename="$(find lms1xx)/urdf/sick_lms1xx_mount.urdf.xacro" /-->
+    <!-- Import camera-->
+    <!--xacro:include filename="$(find realsense_gazebo_plugin)/urdf/realsense-RS200.macro.xacro"/-->
+    <xacro:include filename="$(find mobiman_simulation)/urdf/realsense-d435.macro.xacro" />
+    <!-- Attach robotic arm to the mobile base -->
     <joint name="ur5_to_jackal" type="fixed">
         <parent link="base_link"/>
@@ -24,30 +24,197 @@
         <origin xyz="0 0 0.2" rpy="0 0 0" />
     </joint>
-    <!-- Import macro for lidar-->
-    <xacro:include filename="$(find lms1xx)/urdf/sick_lms1xx_mount.urdf.xacro" />
     <!-- Create lidar instance -->
-  <!--xacro:sick_lms1xx_mount prefix="jackal"
-      parent_link="base_link"
-      topic="jackal/scan"
-      min_range="0.2"
-      max_range="4.0">
-      <origin xyz="0 0 0.18" rpy="0 0 0" />
-  </xacro:sick_lms1xx_mount-->
-    <!-- Import macro for camera-->
-    <!--xacro:include filename="$(find realsense_gazebo_plugin)/urdf/realsense-RS200.macro.xacro"/-->
-    <!--xacro:include filename="$(find tentabot)/urdf/r200.urdf.xacro"/-->
-    <!--xacro:include filename="$(find tentabot)/urdf/realsense-d435.macro.xacro" /-->
-    <!-- Instantiate sensors-->
+    <!--xacro:sick_lms1xx_mount prefix="jackal"
+        parent_link="base_link"
+        topic="jackal/scan"
+        min_range="0.2"
+        max_range="4.0">
+        <origin xyz="0 0 0.18" rpy="0 0 0" />
+    </xacro:sick_lms1xx_mount-->
     <!-- Create camera instance -->
     <!--xacro:realsense-rs200
         prefix="rs200_cam1"
-        parent="$(arg ns)/base_link">
-        <origin xyz="0.0 0.0 0.2" rpy="0.0 0.0 0.0" />
+        parent="top_plate_front_link">
+        <origin xyz="0.0 0.0 0.0" rpy="0.0 0.0 0.0" />
     </xacro:realsense-rs200-->
-    <!-- Create camera instance 1.570796327 (turtlebot3 burger)-->
-    <!--xacro:realsense-d435
+    <!-- Create camera instance -1.570796327 -->
+    <!--xacro:realsense-rs200
+        prefix="rs200_cam2"
+        parent="${arm_prefix}ee_link">
+        <origin xyz="0.0 0.0 -0.05" rpy="0.0 0.0 0.0" />
+    </xacro:realsense-rs200-->
+    <!-- Create camera instance -->
+    <xacro:realsense-d435
         prefix="d435_cam1"
         parent="base_link">
         <origin xyz="0.2 0.0 0.2" rpy="0.0 0.0 0.0" />
+    </xacro:realsense-d435>
+    <!-- Create camera instance -1.570796327 -->
+    <!--xacro:realsense-d435
+        prefix="d435_cam2"
+        parent="${arm_prefix}ee_link">
+        <origin xyz="0.0 0.0 -0.05" rpy="0.0 0.0 0.0" />
     </xacro:realsense-d435-->
+    <!-- Create holonomic virtual links and joints -->
+    <!--link name="virtual_world_link"/>
+    <link name="dummy_link">
+ 	    <inertial>
+            <origin rpy="0.0 0 0" xyz="0 0 0"/>
+            <mass value="0.001" />
+            <inertia ixx="7.58333333333e-07" ixy="0.0" ixz="0.0" iyy="7.58333333333e-07" iyz="0.0" izz="1.25e-06"/>
+        </inertial>
+        <collision>
+            <origin rpy="0.0 0 0" xyz="0 0 0"/>
+            <geometry>
+                <box size="0.01 0.01 0.01"/>
+            </geometry>
+        </collision>
+        <visual>
+            <origin rpy="0.0 0 0" xyz="0 0 0"/>
+            <geometry>
+                <box size="0.01 0.01 0.01"/>
+            </geometry>
+        </visual>
+	</link>
+    <gazebo reference="dummy_link">
+        <mu1>10.0</mu1>
+        <mu2>10.0</mu2>
+        <material>Gazebo/Black</material>
+    </gazebo>
+    <joint name="fixed" type="fixed">
+        <parent link="virtual_world_link"/>
+        <child link="dummy_link"/>
+    </joint>
+    <link name="x_axis_link">
+ 	    <inertial>
+            <origin rpy="0.0 0 0" xyz="0 0 0"/>
+            <mass value="0.001" />
+            <inertia ixx="7.58333333333e-07" ixy="0.0" ixz="0.0" iyy="7.58333333333e-07" iyz="0.0" izz="1.25e-06"/>
+        </inertial>
+        <collision>
+            <origin rpy="0.0 0 0" xyz="0 0 0"/>
+            <geometry>
+                <box size="0.01 0.01 0.01"/>
+            </geometry>
+        </collision>
+        <visual>
+            <origin rpy="0.0 0 0" xyz="0 0 0"/>
+            <geometry>
+                <box size="0.01 0.01 0.01"/>
+            </geometry>
+        </visual>
+	</link>
+    <gazebo reference="x_axis_link">
+        <mu1>10.0</mu1>
+        <mu2>10.0</mu2>
+        <material>Gazebo/Red</material>
+    </gazebo>
+    <joint name="x_axis_joint" type="prismatic">
+        <origin xyz="0 0 0.0" rpy="0.0 0.0 0.0"/>
+        <parent link="dummy_link" />
+        <child link="x_axis_link" />
+        <axis xyz="1 0 0" />
+        <limit effort="0.0001" lower="-20" upper="20" velocity="1" />
+        <dynamics damping="0.00001" friction="1000"/>
+    </joint>
+    <transmission name="tran1">
+        <type>transmission_interface/SimpleTransmission</type>
+        <joint name="x_axis_joint">
+            <hardwareInterface>hardware_interface/EffortJointInterface</hardwareInterface>
+        </joint>
+        <actuator name="motor1">
+            <hardwareInterface>hardware_interface/EffortJointInterface</hardwareInterface>
+            <mechanicalReduction>1</mechanicalReduction>
+        </actuator>
+    </transmission>
+    <link name="y_axis_link">
+ 	    <inertial>
+            <origin rpy="0.0 0 0" xyz="0 0 0"/>
+            <mass value="0.001" />
+            <inertia ixx="7.58333333333e-07" ixy="0.0" ixz="0.0" iyy="7.58333333333e-07" iyz="0.0" izz="1.25e-06"/>
+        </inertial>
+        <collision>
+            <origin rpy="0.0 0 0" xyz="0 0 0"/>
+            <geometry>
+                <box size="0.01 0.01 0.01"/>
+            </geometry>
+        </collision>
+        <visual>
+            <origin rpy="0.0 0 0" xyz="0 0 0"/>
+            <geometry>
+                <box size="0.01 0.01 0.01"/>
+            </geometry>
+        </visual>
+	</link>
+    <gazebo reference="y_axis_link">
+        <mu1>10.0</mu1>
+        <mu2>10.0</mu2>
+        <material>Gazebo/Green</material>
+    </gazebo>
+    <joint name="y_axis_joint" type="prismatic">
+        <origin xyz="0 0 0.0" rpy="0.0 0.0 0.0"/>
+        <parent link="x_axis_link" />
+        <child link="y_axis_link" />
+        <axis xyz="0 1 0" />
+        <limit effort="0.0001" lower="-20" upper="20" velocity="1" />
+        <dynamics damping="0.00001" friction="1000"/>
+    </joint>
+    <transmission name="tran2">
+        <type>transmission_interface/SimpleTransmission</type>
+        <joint name="y_axis_joint">
+            <hardwareInterface>hardware_interface/EffortJointInterface</hardwareInterface>
+        </joint>
+        <actuator name="motor2">
+            <hardwareInterface>hardware_interface/EffortJointInterface</hardwareInterface>
+            <mechanicalReduction>1</mechanicalReduction>
+        </actuator>
+    </transmission>
+    <link name="theta_link">
+ 	    <inertial>
+            <origin rpy="0.0 0 0" xyz="0 0 0"/>
+            <mass value="0.001" />
+            <inertia ixx="7.58333333333e-07" ixy="0.0" ixz="0.0" iyy="7.58333333333e-07" iyz="0.0" izz="1.25e-06"/>
+        </inertial>
+        <collision>
+            <origin rpy="0.0 0 0" xyz="0 0 0"/>
+            <geometry>
+                <box size="0.01 0.01 0.01"/>
+            </geometry>
+        </collision>
+        <visual>
+            <origin rpy="0.0 0 0" xyz="0 0 0"/>
+            <geometry>
+                <box size="0.01 0.01 0.01"/>
+            </geometry>
+        </visual>
+	</link>
+    <gazebo reference="theta_link">
+        <mu1>10.0</mu1>
+        <mu2>10.0</mu2>
+        <material>Gazebo/Blue</material>
+        <self_collide>0</self_collide>
+    </gazebo>
+    <joint name="theta_joint" type="continuous">
+        <origin xyz="0 0 0.0" rpy="0.0 0.0 0.0"/>
+        <parent link="y_axis_link" />
+        <child link="theta_link" />
+        <axis xyz="0 0 1" />
+        <limit effort="0.001" lower="-3.14" upper="3.14" velocity="0.01" />
+        <dynamics damping="0.00001" friction="1000"/>
+    </joint>
+    <transmission name="tran3">
+        <type>transmission_interface/SimpleTransmission</type>
+        <joint name="theta_joint">
+            <hardwareInterface>hardware_interface/EffortJointInterface</hardwareInterface>
+        </joint>
+        <actuator name="motor3">
+            <hardwareInterface>hardware_interface/EffortJointInterface</hardwareInterface>
+            <mechanicalReduction>1</mechanicalReduction>
+        </actuator>
+    </transmission>
+    <joint name="entity_link_joint" type="fixed">
+        <parent link="theta_link"/>
+        <child link="base_link"/>
+        <origin xyz="0 0 0.025" rpy="0 0 0"/>
+    </joint-->
 </robot>

File: mobiman_simulation/urdf/jackal_ur5.urdf (robot description, URDF)
Before this commit: robot jackal_ur5, 23 links, 22 joints
Links:
- removed link ur5_ee_link
- added link d435_cam1camera_bottom_screw_frame
- added link d435_cam1camera_color_frame
- added link d435_cam1camera_color_optical_frame
- added link d435_cam1camera_depth_frame
- added link d435_cam1camera_depth_frame_gazebo
- added link d435_cam1camera_depth_optical_frame
- added link d435_cam1camera_left_ir_frame
- added link d435_cam1camera_left_ir_optical_frame
- added link d435_cam1camera_link, mass 0.180; collision box size=0.02505 0.09 0.025; visual mesh filename=package://mobiman_simulation/meshes/d435.stl scale=0.001 0.001 0.001
- added link d435_cam1camera_right_ir_frame
- added link d435_cam1camera_right_ir_optical_frame
- added link ur5_base_link_inertia, mass 4.0; collision mesh filename=package://ur_description/meshes/ur5/collision/base.stl; visual mesh filename=package://ur_description/meshes/ur5/visual/base.dae
- added link ur5_flange
- link ur5_base_link: mass 4.0 -> None; geometry 
Joints:
- removed joint ur5_ee_fixed_joint
- removed joint ur5_wrist_3_link-tool0_fixed_joint
- added joint d435_cam1camera_color_joint: type fixed, parent d435_cam1camera_depth_frame, child d435_cam1camera_color_frame, origin xyz=0 0.015 0 rpy=0 0 0
- added joint d435_cam1camera_color_optical_joint: type fixed, parent d435_cam1camera_color_frame, child d435_cam1camera_color_optical_frame, origin xyz=0 0 0 rpy=-1.570796327 0 -1.570796327
- added joint d435_cam1camera_depth_joint: type fixed, parent d435_cam1camera_link, child d435_cam1camera_depth_frame, origin xyz=0 0 0 rpy=0 0 0
- added joint d435_cam1camera_depth_optical_joint: type fixed, parent d435_cam1camera_depth_frame, child d435_cam1camera_depth_optical_frame, origin xyz=0 0 0 rpy=-1.570796327 0 -1.570796327
- added joint d435_cam1camera_joint: type fixed, parent base_link, child d435_cam1camera_bottom_screw_frame, origin xyz=0.2 0.0 0.2 rpy=0.0 0.0 0.0
- added joint d435_cam1camera_left_ir_joint: type fixed, parent d435_cam1camera_depth_frame, child d435_cam1camera_left_ir_frame, origin xyz=0 0.0 0 rpy=0 0 0
- added joint d435_cam1camera_left_ir_optical_joint: type fixed, parent d435_cam1camera_left_ir_frame, child d435_cam1camera_left_ir_optical_frame, origin xyz=0 0 0 rpy=-1.570796327 0 -1.570796327
- added joint d435_cam1camera_link_joint: type fixed, parent d435_cam1camera_bottom_screw_frame, child d435_cam1camera_link, origin xyz=0 0.0175 0.0125 rpy=0 0 0
- added joint d435_cam1camera_right_ir_joint: type fixed, parent d435_cam1camera_depth_frame, child d435_cam1camera_right_ir_frame, origin xyz=0 -0.05 0 rpy=0 0 0
- added joint d435_cam1camera_right_ir_optical_joint: type fixed, parent d435_cam1camera_right_ir_frame, child d435_cam1camera_right_ir_optical_frame, origin xyz=0 0 0 rpy=-1.570796327 0 -1.570796327
- added joint d435_cam1gazebo_joint: type fixed, parent d435_cam1camera_link, child d435_cam1camera_depth_frame_gazebo, origin xyz=0 0 0 rpy=-1.570796327 0 -1.570796327
- added joint ur5_base_link-base_link_inertia: type fixed, parent ur5_base_link, child ur5_base_link_inertia, origin xyz=0 0 0 rpy=0 0 3.141592653589793
- added joint ur5_flange-tool0: type fixed, parent ur5_flange, child ur5_tool0, origin xyz=0 0 0 rpy=1.5707963267948966 0 1.5707963267948966
- added joint ur5_wrist_3-flange: type fixed, parent ur5_wrist_3_link, child ur5_flange, origin xyz=0 0 0 rpy=0 -1.5707963267948966 -1.5707963267948966
- joint front_left_wheel: origin xyz=0.131 0.187795 0.0345 rpy=0 0 0 -> xyz=0.131 0.19 0.0345 rpy=0 0 0; type fixed -> continuous
- joint front_right_wheel: origin xyz=0.131 -0.187795 0.0345 rpy=0 0 0 -> xyz=0.131 -0.19 0.0345 rpy=0 0 0; type fixed -> continuous
- joint rear_left_wheel: origin xyz=-0.131 0.187795 0.0345 rpy=0 0 0 -> xyz=-0.131 0.19 0.0345 rpy=0 0 0; type fixed -> continuous
- joint rear_right_wheel: origin xyz=-0.131 -0.187795 0.0345 rpy=0 0 0 -> xyz=-0.131 -0.19 0.0345 rpy=0 0 0; type fixed -> continuous
- joint ur5_base_link-base_fixed_joint: origin xyz=0 0 0 rpy=0 0 -3.141592653589793 -> xyz=0 0 0 rpy=0 0 3.141592653589793
- joint ur5_elbow_joint: axis 0 1 0 -> 0 0 1; limit lower=-3.141592653589793 upper=3.141592653589793 effort=150.0 velocity=3.15 -> lower=-3.141592653589793 upper=3.141592653589793 effort=150.0 velocity=3.141592653589793; origin xyz=0.0 -0.1197 0.425 rpy=0.0 0.0 0.0 -> xyz=-0.425 0 0 rpy=0 0 0
- joint ur5_shoulder_lift_joint: axis 0 1 0 -> 0 0 1; limit lower=-3.141592653589793 upper=3.141592653589793 effort=150.0 velocity=3.15 -> lower=-6.283185307179586 upper=6.283185307179586 effort=150.0 velocity=3.141592653589793; origin xyz=0.0 0.13585 0.0 rpy=0.0 1.5707963267948966 0.0 -> xyz=0 0 0 rpy=1.570796327 0 0
- joint ur5_shoulder_pan_joint: limit lower=-3.141592653589793 upper=3.141592653589793 effort=150.0 velocity=3.15 -> lower=-6.283185307179586 upper=6.283185307179586 effort=150.0 velocity=3.141592653589793; origin xyz=0.0 0.0 0.089159 rpy=0.0 0.0 0.0 -> xyz=0 0 0.089159 rpy=0 0 0; parent ur5_base_link -> ur5_base_link_inertia
- joint ur5_wrist_1_joint: axis 0 1 0 -> 0 0 1; limit lower=-3.141592653589793 upper=3.141592653589793 effort=28.0 velocity=3.2 -> lower=-6.283185307179586 upper=6.283185307179586 effort=28.0 velocity=3.141592653589793; origin xyz=0.0 0.0 0.39225 rpy=0.0 1.5707963267948966 0.0 -> xyz=-0.39225 0 0.10915 rpy=0 0 0
- joint ur5_wrist_2_joint: limit lower=-3.141592653589793 upper=3.141592653589793 effort=28.0 velocity=3.2 -> lower=-6.283185307179586 upper=6.283185307179586 effort=28.0 velocity=3.141592653589793; origin xyz=0.0 0.093 0.0 rpy=0.0 0.0 0.0 -> xyz=0 -0.09465 -1.941303950897609e-11 rpy=1.570796327 0 0
- joint ur5_wrist_3_joint: axis 0 1 0 -> 0 0 1; limit lower=-3.141592653589793 upper=3.141592653589793 effort=28.0 velocity=3.2 -> lower=-6.283185307179586 upper=6.283185307179586 effort=28.0 velocity=3.141592653589793; origin xyz=0.0 0.0 0.09465 rpy=0.0 0.0 0.0 -> xyz=0 0.0823 -1.688001216681175e-11 rpy=1.570796326589793 3.141592653589793 3.141592653589793

Commit message: Minor updates.

File: mobiman_simulation/urdf/jackal_fixedWheel.urdf.xacro (robot description, xacro)
@@ -50,5 +50,5 @@
       <fdir1 value="1 0 0"/>
     </gazebo>
-    <joint name="${prefix}_wheel" type="continuous">
+    <joint name="${prefix}_wheel" type="fixed">
       <parent link="chassis_link"/>
       <child link="${prefix}_wheel_link" />

File: mobiman_simulation/urdf/jackal_fixedWheel_ur5.urdf (robot description, URDF)
Before this commit: robot mobiman, 35 links, 34 joints
Joints:
- joint front_left_wheel: origin xyz=0.131 0.187795 0.0345 rpy=0 0 0 -> xyz=0.131 0.19 0.0345 rpy=0 0 0; type continuous -> fixed
- joint front_right_wheel: origin xyz=0.131 -0.187795 0.0345 rpy=0 0 0 -> xyz=0.131 -0.19 0.0345 rpy=0 0 0; type continuous -> fixed
- joint rear_left_wheel: origin xyz=-0.131 0.187795 0.0345 rpy=0 0 0 -> xyz=-0.131 0.19 0.0345 rpy=0 0 0; type continuous -> fixed
- joint rear_right_wheel: origin xyz=-0.131 -0.187795 0.0345 rpy=0 0 0 -> xyz=-0.131 -0.19 0.0345 rpy=0 0 0; type continuous -> fixed

Commit message: Updated ocs2_mobile_manipulator_mrt_gazebo, ocs2_mrt_loop: Mobile mp can be done using actual state obs from gazebo. TODO: Visualized target is based on the estimated trajectory from the mpc which causes a drift from the actual state of the robot.

File: mobiman_simulation/urdf/jackal_fixedWheel.urdf.xacro (robot description, xacro)
@@ -103,5 +103,5 @@
       <!-- Center of mass -->
       <origin xyz="0.012  0.002 0.067" rpy="0 0 0"/>
-      <mass value="16.523"/>
+      <mass value="160.523"/> <!-- Default: 16.523 -->
       <!-- Moments of inertia: ( chassis without wheels ) -->
       <inertia

File: mobiman_simulation/urdf/jackal_fixedWheel_ur5.urdf (robot description, URDF)
Before this commit: robot mobiman, 35 links, 34 joints
Links:
- link chassis_link: mass 16.523 -> 160.523
