Commit message: Added map_utility and map_utiiity server: compiling. Added world2oct.sh, world2dae.py, blend_convert_to_obj.py: to convert gazebo world to octomap data. It is not working for v1.7 gazebo (recent) and probably going to be deprecated. Updated realsense-d435.macro.xacro: added turnGravity parameter for scanner. Added scanner.launch, scanner_camera_process.launch, scanner_display.launch, scanner.rviz, scanner.urdf.xacro: to scan gazebo objects and keep their pointcloud and respective pose (wrt world).

File: mobiman_simulation/urdf/realsense-d435.macro.xacro (robot description, xacro)
@@ -32,4 +32,5 @@
         <xacro:property name="d435_cam_depth_py" value="0.0175"/>
         <xacro:property name="d435_cam_depth_pz" value="${d435_cam_height/2}"/>
+        <xacro:property name="gravityOff" value="true"/>
         <joint name="${prefix}camera_joint" type="fixed">
             <parent link="${parent}"/>
@@ -40,5 +41,5 @@
         <link name="${prefix}camera_bottom_screw_frame"/>
         <gazebo reference="${prefix}camera_bottom_screw_frame">
-            <turnGravityOff>false</turnGravityOff>
+            <turnGravityOff>${gravityOff}</turnGravityOff>
         </gazebo>
         <joint name="${prefix}camera_link_joint" type="fixed">
@@ -68,5 +69,5 @@
         </link>
         <gazebo reference="${prefix}camera_link">
-            <turnGravityOff>false</turnGravityOff>
+            <turnGravityOff>${gravityOff}</turnGravityOff>
             <material>Gazebo/Grey</material>
         </gazebo>
@@ -79,5 +80,5 @@
         <link name="${prefix}camera_depth_frame"/>
         <gazebo reference="${prefix}camera_depth_frame">
-            <turnGravityOff>false</turnGravityOff>
+            <turnGravityOff>${gravityOff}</turnGravityOff>
         </gazebo>
         <joint name="${prefix}camera_depth_optical_joint" type="fixed">
@@ -88,5 +89,5 @@
         <link name="${prefix}camera_depth_optical_frame"/>
         <gazebo reference="${prefix}camera_depth_optical_frame">
-            <turnGravityOff>false</turnGravityOff>
+            <turnGravityOff>${gravityOff}</turnGravityOff>
         </gazebo>
         <!-- camera left IR joints and links -->
@@ -98,5 +99,5 @@
         <link name="${prefix}camera_left_ir_frame"/>
         <gazebo reference="${prefix}camera_left_ir_frame">
-            <turnGravityOff>false</turnGravityOff>
+            <turnGravityOff>${gravityOff}</turnGravityOff>
         </gazebo>
         <joint name="${prefix}camera_left_ir_optical_joint" type="fixed">
@@ -107,5 +108,5 @@
         <link name="${prefix}camera_left_ir_optical_frame"/>
         <gazebo reference="${prefix}camera_left_ir_optical_frame">
-            <turnGravityOff>false</turnGravityOff>
+            <turnGravityOff>${gravityOff}</turnGravityOff>
         </gazebo>
         <!-- camera right IR joints and links -->
@@ -117,5 +118,5 @@
         <link name="${prefix}camera_right_ir_frame"/>
         <gazebo reference="${prefix}camera_right_ir_frame">
-            <turnGravityOff>false</turnGravityOff>
+            <turnGravityOff>${gravityOff}</turnGravityOff>
         </gazebo>
         <joint name="${prefix}camera_right_ir_optical_joint" type="fixed">
@@ -126,5 +127,5 @@
         <link name="${prefix}camera_right_ir_optical_frame"/>
         <gazebo reference="${prefix}camera_right_ir_optical_frame">
-            <turnGravityOff>false</turnGravityOff>
+            <turnGravityOff>${gravityOff}</turnGravityOff>
         </gazebo>
         <!-- camera color joints and links -->
@@ -136,5 +137,5 @@
         <link name="${prefix}camera_color_frame"/>
         <gazebo reference="${prefix}camera_color_frame">
-            <turnGravityOff>false</turnGravityOff>
+            <turnGravityOff>${gravityOff}</turnGravityOff>
         </gazebo>
         <joint name="${prefix}camera_color_optical_joint" type="fixed">
@@ -145,5 +146,5 @@
         <link name="${prefix}camera_color_optical_frame"/>
         <gazebo reference="${prefix}camera_color_optical_frame">
-            <turnGravityOff>false</turnGravityOff>
+            <turnGravityOff>${gravityOff}</turnGravityOff>
         </gazebo>
         <link name="${prefix}camera_depth_frame_gazebo"/>
@@ -154,5 +155,5 @@
         </joint>
         <gazebo reference="camera_depth_frame_gazebo">
-            <turnGravityOff>false</turnGravityOff>
+            <turnGravityOff>${gravityOff}</turnGravityOff>
         </gazebo>
         <gazebo reference="${prefix}camera_link">
