Commit message: Added pointcloud of scanned objects.Updated gazebo.launch: camera process if removed. Updated jackal_ur5.urdf.xacro: camera is removed. Updated jackal_fixedWheel_ur5.urdf: camera is removed. Updated task_jackal_ur5: added joints to removeJoints but it is not working. NOTE: usePreComputation: false is not working. Might related to urdfs. TODO: Make removeJoints work instead of manually make fixed wheels in urdf.

File: mobiman_simulation/urdf/jackal_ur5.urdf (robot description, URDF)
Before this commit: robot mobiman, 24 links, 23 joints
Links:
- added link d435_cam1camera_bottom_screw_frame
- added link d435_cam1camera_color_frame
- added link d435_cam1camera_color_optical_frame
- added link d435_cam1camera_depth_frame
- added link d435_cam1camera_depth_frame_gazebo
- added link d435_cam1camera_depth_optical_frame
- added link d435_cam1camera_left_ir_frame
- added link d435_cam1camera_left_ir_optical_frame
- added link d435_cam1camera_link, mass 0.180; collision box size=0.02505 0.09 0.025; visual mesh filename=package://mobiman_simulation/meshes/d435.stl scale=0.001 0.001 0.001
- added link d435_cam1camera_right_ir_frame
- added link d435_cam1camera_right_ir_optical_frame
Joints:
- added joint d435_cam1camera_color_joint: type fixed, parent d435_cam1camera_depth_frame, child d435_cam1camera_color_frame, origin xyz=0 0.015 0 rpy=0 0 0
- added joint d435_cam1camera_color_optical_joint: type fixed, parent d435_cam1camera_color_frame, child d435_cam1camera_color_optical_frame, origin xyz=0 0 0 rpy=-1.570796327 0 -1.570796327
- added joint d435_cam1camera_depth_joint: type fixed, parent d435_cam1camera_link, child d435_cam1camera_depth_frame, origin xyz=0 0 0 rpy=0 0 0
- added joint d435_cam1camera_depth_optical_joint: type fixed, parent d435_cam1camera_depth_frame, child d435_cam1camera_depth_optical_frame, origin xyz=0 0 0 rpy=-1.570796327 0 -1.570796327
- added joint d435_cam1camera_joint: type fixed, parent base_link, child d435_cam1camera_bottom_screw_frame, origin xyz=0.2 0.0 0.2 rpy=0.0 0.0 0.0
- added joint d435_cam1camera_left_ir_joint: type fixed, parent d435_cam1camera_depth_frame, child d435_cam1camera_left_ir_frame, origin xyz=0 0.0 0 rpy=0 0 0
- added joint d435_cam1camera_left_ir_optical_joint: type fixed, parent d435_cam1camera_left_ir_frame, child d435_cam1camera_left_ir_optical_frame, origin xyz=0 0 0 rpy=-1.570796327 0 -1.570796327
- added joint d435_cam1camera_link_joint: type fixed, parent d435_cam1camera_bottom_screw_frame, child d435_cam1camera_link, origin xyz=0 0.0175 0.0125 rpy=0 0 0
- added joint d435_cam1camera_right_ir_joint: type fixed, parent d435_cam1camera_depth_frame, child d435_cam1camera_right_ir_frame, origin xyz=0 -0.05 0 rpy=0 0 0
- added joint d435_cam1camera_right_ir_optical_joint: type fixed, parent d435_cam1camera_right_ir_frame, child d435_cam1camera_right_ir_optical_frame, origin xyz=0 0 0 rpy=-1.570796327 0 -1.570796327
- added joint d435_cam1gazebo_joint: type fixed, parent d435_cam1camera_link, child d435_cam1camera_depth_frame_gazebo, origin xyz=0 0 0 rpy=-1.570796327 0 -1.570796327
- joint front_left_wheel: type fixed -> continuous
- joint front_right_wheel: type fixed -> continuous
- joint rear_left_wheel: type fixed -> continuous
- joint rear_right_wheel: type fixed -> continuous

File: mobiman_simulation/urdf/jackal_ur5.urdf.xacro (robot description, xacro)
@@ -17,5 +17,5 @@
     <!-- Import camera-->
     <!--xacro:include filename="$(find realsense_gazebo_plugin)/urdf/realsense-RS200.macro.xacro"/-->
-    <xacro:include filename="$(find mobiman_simulation)/urdf/realsense-d435.macro.xacro" />
+    <!--xacro:include filename="$(find mobiman_simulation)/urdf/realsense_d435.macro.xacro" /-->
     <!-- Attach robotic arm to the mobile base -->
     <joint name="ur5_to_jackal" type="fixed">
@@ -45,9 +45,9 @@
     </xacro:realsense-rs200-->
     <!-- Create camera instance -->
-    <xacro:realsense-d435
+    <!--xacro:realsense-d435
         prefix="d435_cam1"
         parent="base_link">
         <origin xyz="0.2 0.0 0.2" rpy="0.0 0.0 0.0" />
-    </xacro:realsense-d435>
+    </xacro:realsense-d435-->
     <!-- Create camera instance -1.570796327 -->
     <!--xacro:realsense-d435
