Commit message: Added scan_gazebo.launch: launches 4 cams and object of interest(ooi) to scan. Added scanner.launch: saving pointcloud of ooi. Updated map_utility: added gazeboModelCallback which subscribe gazebo models and publish pointclouds of oois. Added map_server (src and launch): initialize map utility object which calls gazeboModelCallback.

File: mobiman_simulation/urdf/conveyor_belt.urdf.xacro (robot description, xacro)
@@ -1,27 +1,15 @@
 <?xml version="1.0"?>
-<robot name="conveyor_gazebo" xmlns:xacro="http://www.ros.org/wiki/xacro">
+<robot name="conveyor_belt" xmlns:xacro="http://www.ros.org/wiki/xacro">
     <xacro:property name="prefix" value="belt" />
     <xacro:property name="parent_link" value="world" />
-    <xacro:property name="x_wrt_parent" value="0.0" />
-    <xacro:property name="y_wrt_parent" value="0.0" />
-    <xacro:property name="z_wrt_parent" value="0.0" />
-    <xacro:property name="roll_wrt_parent" value="0.0" />
-    <xacro:property name="pitch_wrt_parent" value="0.0" />
-    <xacro:property name="yaw_wrt_parent" value="0.0" />
     <xacro:property name="conveyor_size_x" value="10.0" />
     <xacro:property name="conveyor_size_y" value="0.5" />
     <xacro:property name="conveyor_size_z" value="0.2" />
-    <xacro:property name="conveyor_pos_x" value="0.0" />
-    <xacro:property name="conveyor_pos_y" value="0.0" />
-    <xacro:property name="conveyor_pos_z" value="0.05" />
+    <xacro:property name="moving_gap_x" value="0.0" />
+    <xacro:property name="moving_gap_y" value="0.0" />
+    <xacro:property name="moving_gap_z" value="0.05" />
     <xacro:property name="PI" value="3.1415926535897931" />
     <xacro:macro name="conveyor_belt" params="prefix
                                               parent_link
-                                              x_wrt_parent
-                                              y_wrt_parent
-                                              z_wrt_parent
-                                              roll_wrt_parent
-                                              pitch_wrt_parent
-                                              yaw_wrt_parent
                                               conveyor_size_x
                                               conveyor_size_y
@@ -30,6 +18,6 @@
             <parent link="${parent_link}"/>
             <child link="${prefix}_visual"/>
-            <origin xyz="${x_wrt_parent} ${y_wrt_parent} ${z_wrt_parent + conveyor_size_z / 2}"
-                    rpy="${roll_wrt_parent} ${pitch_wrt_parent} ${yaw_wrt_parent}" />
+            <origin xyz="0.0 0.0 0.0"
+                    rpy="0.0 0.0 0.0" />
         </joint>
         <link name="${prefix}_visual">
@@ -66,5 +54,5 @@
             </inertial>
             <collision>
-                <origin xyz="${conveyor_pos_x} ${conveyor_pos_y} ${conveyor_pos_z}" rpy="0 0 0"/>
+                <origin xyz="${moving_gap_x} ${moving_gap_y} ${moving_gap_z}" rpy="0 0 0"/>
                 <geometry>
                     <box size="${conveyor_size_x} ${conveyor_size_y} ${conveyor_size_z}"/>
@@ -73,9 +61,9 @@
         </link>
         <joint name="belt_joint" type="prismatic">
-            <origin xyz="0.0 0.0 0.05" rpy="0 0 0"/>
+            <origin xyz="0.0 0.0 0.0" rpy="0 0 0"/>
             <parent link="${prefix}_visual"/>
             <child link="${prefix}_moving"/>
             <axis xyz="1 0 0"/>
-            <limit lower="0.0" upper="1.0" effort="1000" velocity="1000"/>
+            <limit lower="0.0" upper="1.0" effort="100" velocity="100"/>
         </joint>
         <gazebo>
@@ -92,10 +80,4 @@
     <xacro:conveyor_belt prefix="${prefix}"
                          parent_link="${parent_link}"
-                         x_wrt_parent="${x_wrt_parent}"
-                         y_wrt_parent="${y_wrt_parent}"
-                         z_wrt_parent="${z_wrt_parent}"
-                         roll_wrt_parent="${roll_wrt_parent}"
-                         pitch_wrt_parent="${pitch_wrt_parent}"
-                         yaw_wrt_parent="${yaw_wrt_parent}"
                          conveyor_size_x="${conveyor_size_x}"
                          conveyor_size_y="${conveyor_size_y}"

File: mobiman_simulation/urdf/dep/conveyor.urdf (robot description, URDF)
Before this commit: robot conveyor_gazebo, 3 links, 2 joints
Joints:
- joint belt_joint: origin xyz=0.0 0.0 0.05 rpy=0 0 0 -> xyz=0.0 0.0 0.0 rpy=0 0 0
- joint fixed: origin xyz=0.0 0.0 0.1 rpy=0.0 0.0 0.0 -> xyz=0.0 0.0 0.0 rpy=0.0 0.0 0.0

File: mobiman_simulation/urdf/scanner.urdf.xacro (robot description, xacro)
@@ -8,5 +8,5 @@
     <xacro:include filename="$(find mobiman_simulation)/urdf/materials.xacro" />
     <!-- Import camera-->
-    <xacro:include filename="$(find mobiman_simulation)/urdf/realsense-d435.macro.xacro" />
+    <xacro:include filename="$(find mobiman_simulation)/urdf/realsense_d435_gravityOff.macro.xacro" />
     <link name="base_link"></link>
     <!-- Create camera instance (1.0 1.0 1.0) -->
