Commit message: Updated map_utility, scanner, map_server: pc2 of actors are scanned and added into octomap. Tested, working successfully. NOTE: There are jitters while actors are moving in octomap!

File: mobiman_simulation/urdf/package.urdf.xacro (robot description, xacro)
@@ -5,4 +5,5 @@
     <material name="Green"><color rgba="0 1 0 1"/></material>
     <material name="Blue"><color rgba="0 0 1 1"/></material>
+    <material name="White"><color rgba="1 1 1 1"/></material>
     <xacro:macro name="package" params="prefix
                                         color
