Commit message: Updated red_cube.urdf, red_cube.urdf.xacro: reduced mass to 0.1.

File: mobiman_simulation/urdf/red_cube.urdf (robot description, URDF)
Before this commit: robot red_cube_gazebo, 1 links, 0 joints
Links:
- link red_cube_base_link: mass 0.2 -> 0.1

File: mobiman_simulation/urdf/red_cube.urdf.xacro (robot description, xacro)
@@ -6,5 +6,5 @@
         prefix="red_cube"
         color="Red"
-        mass="0.2"
+        mass="0.1"
         box_size_x="0.05"
         box_size_y="0.05"
