Commit message: Added ocs2 data for debugging joint limit issue. Updated plot_ocs2_log: extracting and plotting individual logs and log in folder. Individual is working well but extract_and_plot_log_in_folder function needs to be debugged, since the data seems like concatenating wrong (y is getting when logs are concatenated).

File: mobiman_simulation/urdf/jackal_fixedWheel_jaco_fixedFinger.urdf (robot description, URDF)
Before this commit: robot mobiman, 39 links, 38 joints
Joints:
- joint j2n6s300_joint_1: limit lower=-300 upper=300 effort=40 velocity=0.6283185307179586 -> lower=-628.3185307179587 upper=628.3185307179587 effort=40 velocity=0.6283185307179586
- joint j2n6s300_joint_4: limit lower=-300 upper=300 effort=20 velocity=0.8377580409572781 -> lower=-628.3185307179587 upper=628.3185307179587 effort=20 velocity=0.8377580409572781
- joint j2n6s300_joint_5: limit lower=-300 upper=300 effort=20 velocity=0.8377580409572781 -> lower=-628.3185307179587 upper=628.3185307179587 effort=20 velocity=0.8377580409572781
- joint j2n6s300_joint_6: limit lower=-300 upper=300 effort=20 velocity=0.8377580409572781 -> lower=-628.3185307179587 upper=628.3185307179587 effort=20 velocity=0.8377580409572781
