Commit message: fix-urdf-cleanup-reset

File: mobiman_simulation/urdf/jackal_jaco.urdf (robot description, URDF)
Before this commit: robot mobiman, 39 links, 38 joints
Links:
- removed link j2n6s300_link_finger_1
- removed link j2n6s300_link_finger_2
- removed link j2n6s300_link_finger_3
- removed link j2n6s300_link_finger_tip_1
- removed link j2n6s300_link_finger_tip_2
- removed link j2n6s300_link_finger_tip_3
Joints:
- removed joint j2n6s300_joint_finger_1
- removed joint j2n6s300_joint_finger_2
- removed joint j2n6s300_joint_finger_3
- removed joint j2n6s300_joint_finger_tip_1
- removed joint j2n6s300_joint_finger_tip_2
- removed joint j2n6s300_joint_finger_tip_3
- joint j2n6s300_joint_1: origin xyz=0 0 0.15675 rpy=0 3.141592653589793 0 -> xyz=0 0 0.16075 rpy=0 3.141592653589793 0

Commit message: fix-urdf

File: mobiman_simulation/urdf/jackal_jaco.urdf (robot description, URDF)
Before this commit: robot mobiman, 33 links, 32 joints
Joints:
- joint j2n6s300_joint_1: origin xyz=0 0 0.16075 rpy=0 3.141592653589793 0 -> xyz=0 0 0.16575 rpy=0 3.141592653589793 0

Commit message: Updated jackal_jaco.urdf: still issues while re-spawning in gazebo. Updated plot_functions: not all reward functions are plotted yet.

File: mobiman_simulation/urdf/jackal_jaco.urdf (robot description, URDF)
Before this commit: robot mobiman, 33 links, 32 joints
Joints:
- joint j2n6s300_joint_1: origin xyz=0 0 0.16575 rpy=0 3.141592653589793 0 -> xyz=0 0 0.16975 rpy=0 3.141592653589793 0
