Commit message: Updated conveyor_belt.urdf, conveyor_belt.urdf.xacro, conveyor_belt.json: conveyor belt width is decreased to decrease the collision chance during manipulation.

File: mobiman_simulation/urdf/conveyor_belt.urdf (robot description, URDF)
Before this commit: robot conveyor_belt, 3 links, 2 joints
Links:
- link belt_moving: geometry collision box size=10.0 0.18 0.4
- link belt_visual: geometry collision box size=10.0 0.18 0.4; visual box size=10.0 0.18 0.4

File: mobiman_simulation/urdf/conveyor_belt.urdf.xacro (robot description, xacro)
@@ -4,6 +4,6 @@
     <xacro:property name="parent_link" value="world" />
     <xacro:property name="conveyor_size_x" value="10.0" />
-    <xacro:property name="conveyor_size_y" value="0.5" />
-    <xacro:property name="conveyor_size_z" value="0.2" />
+    <xacro:property name="conveyor_size_y" value="0.18" />
+    <xacro:property name="conveyor_size_z" value="0.4" />
     <xacro:property name="moving_gap_x" value="0.0" />
     <xacro:property name="moving_gap_y" value="0.0" />

Commit message: Updated conveyor_belt.urdf.xacro, conveyor_belt.urdf: increased the mass to 20kg.

File: mobiman_simulation/urdf/conveyor_belt.urdf (robot description, URDF)
Before this commit: robot conveyor_belt, 3 links, 2 joints
Links:
- link belt_moving: mass 1 -> 20
- link belt_visual: mass 1 -> 20

File: mobiman_simulation/urdf/conveyor_belt.urdf.xacro (robot description, xacro)
@@ -37,5 +37,5 @@
             <inertial>
                 <origin xyz="0.0 0.0 0.0" rpy="0 0 0"/>
-                <mass value="1"/>
+                <mass value="20"/>
                 <inertia
                     ixx="1.0" ixy="0.0" ixz="0.0"
@@ -47,5 +47,5 @@
             <inertial>
                 <origin xyz="0.0 0.0 0.0" rpy="0 0 0"/>
-                <mass value="1"/>
+                <mass value="20"/>
                 <inertia
                     ixx="1.0" ixy="0.0" ixz="0.0"

Commit message: Updated urfd and point cloud data of red_cube and conveyor.

File: mobiman_simulation/urdf/conveyor_belt.urdf (robot description, URDF)
Before this commit: robot conveyor_belt, 3 links, 2 joints
Links:
- link belt_moving: geometry collision box size=2.0 0.35 0.5
- link belt_visual: geometry collision box size=2.0 0.35 0.5; visual box size=2.0 0.35 0.5

File: mobiman_simulation/urdf/conveyor_belt.urdf.xacro (robot description, xacro)
@@ -3,7 +3,7 @@
     <xacro:property name="prefix" value="belt" />
     <xacro:property name="parent_link" value="world" />
-    <xacro:property name="conveyor_size_x" value="10.0" />
-    <xacro:property name="conveyor_size_y" value="0.18" />
-    <xacro:property name="conveyor_size_z" value="0.4" />
+    <xacro:property name="conveyor_size_x" value="2.0" />
+    <xacro:property name="conveyor_size_y" value="0.35" />
+    <xacro:property name="conveyor_size_z" value="0.5" />
     <xacro:property name="moving_gap_x" value="0.0" />
     <xacro:property name="moving_gap_y" value="0.0" />

File: mobiman_simulation/urdf/red_cube.urdf (robot description, URDF)
Before this commit: robot red_cube_gazebo, 1 links, 0 joints
Links:
- link red_cube_base_link: geometry collision box size=0.15 0.075 0.15; visual box size=0.15 0.075 0.15

File: mobiman_simulation/urdf/red_cube.urdf.xacro (robot description, xacro)
@@ -7,7 +7,7 @@
         color="Red"
         mass="0.1"
-        box_size_x="0.05"
-        box_size_y="0.05"
-        box_size_z="0.05" >
+        box_size_x="0.15"
+        box_size_y="0.075"
+        box_size_z="0.15" >
     </xacro:package>
 </robot>
