Commit message: Updated gazebo.launch: no init robot pose, kept same with urdf. Updated jackal_fixedWheel_ur5: robot initial pose is updated through URDF.

File: mobiman_simulation/urdf/dep/jackal_fixedWheel_ur5_dep.urdf (robot description, URDF)
Before this commit: robot mobiman, 35 links, 34 joints
Joints:
- joint front_left_wheel: origin xyz=0.131 0.187795 0.0345 rpy=0 0 0 -> xyz=0.131 0.19 0.0345 rpy=0 0 0
- joint front_right_wheel: origin xyz=0.131 -0.187795 0.0345 rpy=0 0 0 -> xyz=0.131 -0.19 0.0345 rpy=0 0 0
- joint rear_left_wheel: origin xyz=-0.131 0.187795 0.0345 rpy=0 0 0 -> xyz=-0.131 0.19 0.0345 rpy=0 0 0
- joint rear_right_wheel: origin xyz=-0.131 -0.187795 0.0345 rpy=0 0 0 -> xyz=-0.131 -0.19 0.0345 rpy=0 0 0
- joint ur5_elbow_joint: origin xyz=-0.425 0 0 rpy=0 0 -2.0 -> xyz=-0.425 0 0 rpy=0 0 0
- joint ur5_shoulder_pan_joint: origin xyz=0 0 0.089159 rpy=0 0 3.141592653589793 -> xyz=0 0 0.089159 rpy=0 0 0
- joint ur5_wrist_1_joint: origin xyz=-0.39225 0 0.10915 rpy=0 0 3.141592653589793 -> xyz=-0.39225 0 0.10915 rpy=0 0 0
