Commit message: NUA: Commiting changes that Sarvesh did for experiments.

File: mobiman_simulation/urdf/tmp/jackal_jaco.urdf (robot description, URDF)
Before this commit: robot mobiman, 39 links, 38 joints
Joints:
- joint jaco_to_jackal: origin xyz=0 0 0.2 rpy=0 0 0 -> xyz=0.022 -0.078 0.015 rpy=0 0 0
